File: ALU/Simulation/Simulation.kicad_sch (KiCad schematic)
At the start: 2 parts

Commit message: Delete files
Parts:
- removed D?: LED, symbol Device:LED
- removed U?: 74HC04, symbol 74xx:74HC04
- added D? (x4): LED, symbol Device:LED
- added SW_1: SW_DIP_x08, symbol Switch:SW_DIP_x08
- added SW_2: SW_DIP_x03, symbol Switch:SW_DIP_x03
- added U_1: 74157, symbol 74xx_IEEE:74157
- added V?: VSOURCE, symbol pspice:VSOURCE
Connections:
- new net: SW_1.1, SW_1.2, SW_1.3, SW_1.4, SW_1.5, SW_1.6, SW_1.7, SW_1.8, SW_2.1, SW_2.2, SW_2.3, V?.1 (E1)
- new net: D?.2 (A), U_1.4 (Qa)
- new net: D?.2 (A), U_1.7 (Qb)
- new net: SW_2.4, U_1.1 (A/B)
- new net: D?.2 (A), U_1.9 (Qd)
- new net: D?.2 (A), U_1.12 (Qc)
- new net: SW_1.10, U_1.14 (I0c)
- new net: SW_1.11, U_1.5 (I0b)
- new net: SW_1.12, U_1.2 (I0a)
- new net: SW_1.9, U_1.11 (I0d)
- new net +5V: U_1.10 (I1d), U_1.13 (I1c), U_1.15 (~{EN}), U_1.16 (VCC), U_1.3 (I1a), U_1.6 (I1b)
- new net GND: D?.1 (K), D?.1 (K), D?.1 (K), D?.1 (K), SW_1.13, SW_1.14, SW_1.15, SW_1.16, SW_2.5, SW_2.6, U_1.8 (GND), V?.2 (E2)

Commit message: Update Sim try version
Parts:
- gave numbers to parts that had none: 4
Changed lines of the file:
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@@
   (symbol (lib_id "Device:LED") (at 91.44 25.4 180) (unit 1)
     (in_bom yes) (on_board yes) (fields_autoplaced)
-    (property "Reference" "D?" (id 0) (at 93.0275 17.78 0))
+    (property "Reference" "D1" (id 0) (at 93.0275 17.78 0))
     (property "Value" "LED" (id 1) (at 93.0275 20.32 0))
     (property "Footprint" "" (id 2) (at 91.44 25.4 0)
@@
   (symbol (lib_id "Device:LED") (at 91.44 30.48 180) (unit 1)
     (in_bom yes) (on_board yes) (fields_autoplaced)
-    (property "Reference" "D?" (id 0) (at 93.0275 22.86 0))
+    (property "Reference" "D2" (id 0) (at 93.0275 22.86 0))
     (property "Value" "LED" (id 1) (at 93.0275 25.4 0))
     (property "Footprint" "" (id 2) (at 91.44 30.48 0)
@@
   (symbol (lib_id "Device:LED") (at 91.44 40.64 180) (unit 1)
     (in_bom yes) (on_board yes) (fields_autoplaced)
-    (property "Reference" "D?" (id 0) (at 93.0275 33.02 0))
+    (property "Reference" "D4" (id 0) (at 93.0275 33.02 0))
     (property "Value" "LED" (id 1) (at 93.0275 35.56 0))
     (property "Footprint" "" (id 2) (at 91.44 40.64 0)
@@
   (symbol (lib_id "Device:LED") (at 91.44 35.56 180) (unit 1)
     (in_bom yes) (on_board yes) (fields_autoplaced)
-    (property "Reference" "D?" (id 0) (at 93.0275 27.94 0))
+    (property "Reference" "D3" (id 0) (at 93.0275 27.94 0))
     (property "Value" "LED" (id 1) (at 93.0275 30.48 0))
     (property "Footprint" "" (id 2) (at 91.44 35.56 0)
@@
     )
     (path "/3aa836fe-5067-4e7b-8606-0c2c32c78734"
-      (reference "D?") (unit 1) (value "LED") (footprint "")
+      (reference "D1") (unit 1) (value "LED") (footprint "")
     )
     (path "/4ce2d8e4-fdf2-4ddb-9484-341159338b42"
-      (reference "D?") (unit 1) (value "LED") (footprint "")
+      (reference "D2") (unit 1) (value "LED") (footprint "")
+    )
+    (path "/be7bbeda-6f43-4ea3-b62d-b60b842fcfc1"
+      (reference "D3") (unit 1) (value "LED") (footprint "")
     )
     (path "/5c2ff34b-c7c8-4e3f-8f38-fdd9fbee5513"
-      (reference "D?") (unit 1) (value "LED") (footprint "")
-    )
-    (path "/be7bbeda-6f43-4ea3-b62d-b60b842fcfc1"
-      (reference "D?") (unit 1) (value "LED") (footprint "")
+      (reference "D4") (unit 1) (value "LED") (footprint "")
     )
     (path "/c93aa7fc-75c1-4e34-818e-66ed4d7f353a"
